Commit message: feat: 공식 트랙과 단일 모터·ToF 주행 기준선 반영

File: src/arena_description/models/arena_car/model.sdf.xacro (robot description, xacro)
@@ -4,5 +4,34 @@
   <xacro:arg name="body_width" default="0.15"/>
   <xacro:arg name="body_height" default="0.06"/>
-  <xacro:arg name="body_mass" default="1.5"/>
+  <xacro:arg name="body_mass" default="1.635"/>
+  <xacro:arg name="body_cg_z_offset" default="0.0"/>
+  <xacro:arg name="drive_mode" default="single_motor"/>
+  <xacro:arg name="render_sensors" default="true"/>
+  <xacro:arg name="gear_ratio" default="8.0"/>
+  <xacro:arg name="gear_efficiency" default="1.0"/>
+  <xacro:arg name="motor_torque_limit" default="0.060"/>
+  <xacro:arg name="motor_brake_torque_limit" default="0.045"/>
+  <xacro:arg name="motor_free_speed" default="2200.0"/>
+  <xacro:arg name="motor_response_time" default="0.040"/>
+  <xacro:arg name="motor_speed_kp" default="0.10"/>
+  <xacro:arg name="motor_speed_ki" default="0.20"/>
+  <xacro:arg name="motor_acceleration" default="3.0"/>
+  <xacro:arg name="motor_timeout" default="0.5"/>
+  <xacro:arg name="carrier_drag" default="0.0"/>
+  <xacro:arg name="differential_viscosity" default="0.0"/>
+  <xacro:arg name="differential_torque_limit" default="0.0"/>
+  <xacro:arg name="servo_position_gain" default="0.40"/>
+  <xacro:arg name="servo_integral_gain" default="0.25"/>
+  <xacro:arg name="servo_velocity_gain" default="0.003"/>
+  <xacro:arg name="servo_torque_limit" default="0.12"/>
+  <xacro:arg name="servo_rate_limit" default="4.0"/>
+  <xacro:arg name="tire_mu_lateral" default="0.9"/>
+  <xacro:arg name="tire_mu_longitudinal" default="0.9"/>
+  <xacro:arg name="tire_slip_lateral" default="0.02"/>
+  <xacro:arg name="tire_slip_longitudinal" default="0.02"/>
+  <xacro:arg name="tire_normal_force" default="4.905"/>
+  <xacro:arg name="wheel_damping" default="0.000005"/>
+  <!-- 시험용 한쪽 타이어 마찰 배율. 기본값은 좌우 동일합니다. -->
+  <xacro:arg name="rear_left_friction_scale" default="1.0"/>
   <xacro:arg name="wheelbase" default="0.145"/>
   <xacro:arg name="track_width" default="0.135"/>
@@ -10,5 +39,5 @@
   <xacro:arg name="wheel_width" default="0.012"/>
   <xacro:arg name="max_steering_angle" default="0.45"/>
-  <xacro:arg name="max_speed" default="2.0"/>
+  <xacro:arg name="max_speed" default="5.5555555556"/>
   <xacro:arg name="steering_p_gain" default="12.0"/>
   <xacro:arg name="acceleration_limit" default="4.0"/>
@@ -131,6 +160,7 @@
   <xacro:property name="wheel_mass" value="0.04"/>
   <xacro:property name="steering_link_mass" value="0.01"/>
-  <xacro:macro name="box_inertial" params="mass x y z">
+  <xacro:macro name="box_inertial" params="mass x y z cg_z:=0">
     <inertial>
+      <pose>0 0 ${cg_z} 0 0 0</pose>
       <mass>${mass}</mass>
       <inertia>
@@ -157,5 +187,5 @@
     </inertial>
   </xacro:macro>
-  <xacro:macro name="wheel_link" params="name x y">
+  <xacro:macro name="wheel_link" params="name x y friction_scale:=1">
     <link name="${name}">
       <pose>${x} ${y} ${wheel_radius} ${-pi / 2.0} 0 0</pose>
@@ -183,7 +213,8 @@
           <friction>
             <ode>
-              <mu>1.2</mu>
-              <mu2>1.0</mu2>
-              <fdir1>0 1 0</fdir1>
+              <mu>${float('$(arg tire_mu_lateral)') * float(friction_scale)}</mu>
+              <mu2>${float('$(arg tire_mu_longitudinal)') * float(friction_scale)}</mu2>
+              <!-- WheelSlip 규약: 바퀴 로컬 회전축 Z와 평행, 횡방향 마찰. -->
+              <fdir1>0 0 1</fdir1>
             </ode>
           </friction>
@@ -202,6 +233,7 @@
           <upper>1.79769e+308</upper>
           <effort>5.0</effort>
-          <velocity>200.0</velocity>
+          <velocity>1500.0</velocity>
         </limit>
+        <dynamics><damping>$(arg wheel_damping)</damping></dynamics>
       </axis>
     </joint>
@@ -226,4 +258,5 @@
         </material>
       </visual>
+      <xacro:if value="$(arg render_sensors)">
       <sensor name="tof_${name}" type="gpu_lidar">
         <always_on>true</always_on>
@@ -255,4 +288,5 @@
         </lidar>
       </sensor>
+      </xacro:if>
     </link>
     <joint name="tof_${name}_fixed_joint" type="fixed">
@@ -266,5 +300,5 @@
     <link name="chassis">
       <pose>0 0 ${wheel_radius + body_height / 2.0} 0 0 0</pose>
-      <xacro:box_inertial mass="${body_mass}" x="${body_length}" y="${body_width}" z="${body_height}"/>
+      <xacro:box_inertial mass="${body_mass}" x="${body_length}" y="${body_width}" z="${body_height}" cg_z="$(arg body_cg_z_offset)"/>
       <visual name="visual">
         <geometry>
@@ -298,4 +332,5 @@
         </material>
       </visual>
+      <xacro:if value="$(arg render_sensors)">
       <sensor name="d435i_color" type="camera">
         <camera name="color">
@@ -363,4 +398,5 @@
       </sensor>
       </xacro:if>
+      </xacro:if>
       <sensor name="d435i_imu" type="imu">
         <always_on>true</always_on>
@@ -389,4 +425,5 @@
           <material><ambient>0.9 0.27 0.025 1</ambient><diffuse>0.95 0.32 0.03 1</diffuse></material>
         </visual>
+        <xacro:if value="$(arg render_sensors)">
         <sensor name="rplidar_c1" type="gpu_lidar">
           <always_on>true</always_on>
@@ -406,4 +443,5 @@
           </lidar>
         </sensor>
+        </xacro:if>
       </link>
       <joint name="lidar_fixed_joint" type="fixed"><parent>chassis</parent><child>lidar_link</child></joint>
@@ -419,5 +457,5 @@
     <xacro:wheel_link name="front_left_wheel" x="${wheelbase / 2.0}" y="${track_width / 2.0}"/>
     <xacro:wheel_link name="front_right_wheel" x="${wheelbase / 2.0}" y="${-track_width / 2.0}"/>
-    <xacro:wheel_link name="rear_left_wheel" x="${-wheelbase / 2.0}" y="${track_width / 2.0}"/>
+    <xacro:wheel_link name="rear_left_wheel" x="${-wheelbase / 2.0}" y="${track_width / 2.0}" friction_scale="$(arg rear_left_friction_scale)"/>
     <xacro:wheel_link name="rear_right_wheel" x="${-wheelbase / 2.0}" y="${-track_width / 2.0}"/>
     <link name="front_left_steering_link">
@@ -467,4 +505,5 @@
     <xacro:wheel_joint name="rear_left_wheel_joint" parent="chassis" child="rear_left_wheel"/>
     <xacro:wheel_joint name="rear_right_wheel_joint" parent="chassis" child="rear_right_wheel"/>
+    <xacro:if value="${'$(arg drive_mode)' == 'legacy_velocity'}">
     <plugin filename="gz-sim-ackermann-steering-system" name="gz::sim::systems::AckermannSteering">
       <left_joint>rear_left_wheel_joint</left_joint>
@@ -490,4 +529,46 @@
       <child_frame_id>base_link</child_frame_id>
     </plugin>
+    </xacro:if>
+    <xacro:if value="${'$(arg drive_mode)' == 'single_motor'}">
+    <plugin filename="arena-single-motor-system" name="arena::SingleMotorDrive">
+      <wheel_radius>${wheel_radius}</wheel_radius>
+      <wheelbase>${wheelbase}</wheelbase>
+      <track_width>${track_width}</track_width>
+      <steering_limit>${max_steering_angle}</steering_limit>
+      <max_speed>${max_speed}</max_speed>
+      <gear_ratio>$(arg gear_ratio)</gear_ratio>
+      <gear_efficiency>$(arg gear_efficiency)</gear_efficiency>
+      <motor_torque_limit>$(arg motor_torque_limit)</motor_torque_limit>
+      <motor_brake_torque_limit>$(arg motor_brake_torque_limit)</motor_brake_torque_limit>
+      <motor_free_speed>$(arg motor_free_speed)</motor_free_speed>
+      <motor_response_time>$(arg motor_response_time)</motor_response_time>
+      <speed_kp>$(arg motor_speed_kp)</speed_kp>
+      <speed_ki>$(arg motor_speed_ki)</speed_ki>
+      <acceleration_limit>$(arg motor_acceleration)</acceleration_limit>
+      <command_timeout>$(arg motor_timeout)</command_timeout>
+      <carrier_drag>$(arg carrier_drag)</carrier_drag>
+      <differential_viscosity>$(arg differential_viscosity)</differential_viscosity>
+      <differential_torque_limit>$(arg differential_torque_limit)</differential_torque_limit>
+      <steering_gain>$(arg servo_position_gain)</steering_gain>
+      <steering_integral_gain>$(arg servo_integral_gain)</steering_integral_gain>
+      <steering_velocity_gain>$(arg servo_velocity_gain)</steering_velocity_gain>
+      <steering_torque_limit>$(arg servo_torque_limit)</steering_torque_limit>
+      <steering_rate_limit>$(arg servo_rate_limit)</steering_rate_limit>
+    </plugin>
+    <plugin filename="gz-sim-wheel-slip-system" name="gz::sim::systems::WheelSlip">
+      <xacro:macro name="slip_wheel" params="name">
+        <wheel link_name="${name}">
+          <slip_compliance_lateral>$(arg tire_slip_lateral)</slip_compliance_lateral>
+          <slip_compliance_longitudinal>$(arg tire_slip_longitudinal)</slip_compliance_longitudinal>
+          <wheel_normal_force>$(arg tire_normal_force)</wheel_normal_force>
+          <wheel_radius>${wheel_radius}</wheel_radius>
+        </wheel>
+      </xacro:macro>
+      <xacro:slip_wheel name="front_left_wheel"/>
+      <xacro:slip_wheel name="front_right_wheel"/>
+      <xacro:slip_wheel name="rear_left_wheel"/>
+      <xacro:slip_wheel name="rear_right_wheel"/>
+    </plugin>
+    </xacro:if>
     <plugin filename="gz-sim-joint-state-publisher-system" name="gz::sim::systems::JointStatePublisher">
       <topic>/model/arena_car/joint_state</topic>

Commit message: feat: 공식 트랙 v2026.09.02 및 차량 식별 마커 반영

File: src/arena_description/models/arena_car/model.sdf.xacro (robot description, xacro)
@@ -8,4 +8,11 @@
   <xacro:arg name="drive_mode" default="single_motor"/>
   <xacro:arg name="render_sensors" default="true"/>
+  <xacro:arg name="rear_marker_enabled" default="true"/>
+  <xacro:arg name="rear_marker_x" default="-0.1005"/>
+  <xacro:arg name="rear_marker_y" default="0.0"/>
+  <xacro:arg name="rear_marker_z" default="0.090"/>
+  <xacro:arg name="rear_marker_yaw" default="3.1415926536"/>
+  <xacro:arg name="rear_marker_board_size" default="0.050"/>
+  <xacro:arg name="rear_marker_code_size" default="0.035"/>
   <xacro:arg name="gear_ratio" default="8.0"/>
   <xacro:arg name="gear_efficiency" default="1.0"/>
@@ -160,4 +167,5 @@
   <xacro:property name="wheel_mass" value="0.04"/>
   <xacro:property name="steering_link_mass" value="0.01"/>
+  <xacro:property name="rear_marker_cell_size" value="${float('$(arg rear_marker_code_size)') / 6.0}"/>
   <xacro:macro name="box_inertial" params="mass x y z cg_z:=0">
     <inertial>
@@ -295,4 +303,26 @@
     </joint>
   </xacro:macro>
+  <!--
+    팀 시험용 후방 식별 마커: DICT_4X4_50 ID 10. 5 cm 인쇄판 안에
+    3.5 cm 코드를 두어 양쪽 7.5 mm 흰 여백을 확보합니다. 운영진이 사전·ID·
+    설치 위치를 확정하면 교체해야 하며, 현재는 충돌체가 없는 표시용 형상입니다.
+  -->
+  <xacro:macro name="rear_marker_id10_cell" params="row col">
+    <xacro:property name="marker_local_y" value="${-float('$(arg rear_marker_code_size)') / 2.0 + (float(col) + 0.5) * rear_marker_cell_size}"/>
+    <xacro:property name="marker_local_z" value="${float('$(arg rear_marker_code_size)') / 2.0 - (float(row) + 0.5) * rear_marker_cell_size}"/>
+    <visual name="rear_marker_id10_ink_${row}_${col}">
+      <pose>${float('$(arg rear_marker_x)') + 0.0007 * cos(float('$(arg rear_marker_yaw)')) - marker_local_y * sin(float('$(arg rear_marker_yaw)'))}
+            ${float('$(arg rear_marker_y)') + 0.0007 * sin(float('$(arg rear_marker_yaw)')) + marker_local_y * cos(float('$(arg rear_marker_yaw)'))}
+            ${float('$(arg rear_marker_z)') - (wheel_radius + body_height / 2.0) + marker_local_z}
+            0 0 $(arg rear_marker_yaw)</pose>
+      <geometry><box><size>0.0004 ${rear_marker_cell_size} ${rear_marker_cell_size}</size></box></geometry>
+      <material>
+        <ambient>0.002 0.002 0.002 1</ambient>
+        <diffuse>0.002 0.002 0.002 1</diffuse>
+        <specular>0 0 0 1</specular>
+      </material>
+      <cast_shadows>false</cast_shadows>
+    </visual>
+  </xacro:macro>
   <model name="arena_car">
     <self_collide>false</self_collide>
@@ -313,4 +343,30 @@
         </material>
       </visual>
+      <xacro:if value="$(arg rear_marker_enabled)">
+        <visual name="rear_marker_id10_board">
+          <pose>$(arg rear_marker_x) $(arg rear_marker_y)
+                ${float('$(arg rear_marker_z)') - (wheel_radius + body_height / 2.0)}
+                0 0 $(arg rear_marker_yaw)</pose>
+          <geometry><box><size>0.001 $(arg rear_marker_board_size) $(arg rear_marker_board_size)</size></box></geometry>
+          <material>
+            <ambient>1 1 1 1</ambient><diffuse>1 1 1 1</diffuse><specular>0 0 0 1</specular>
+          </material>
+          <cast_shadows>false</cast_shadows>
+        </visual>
+        <xacro:rear_marker_id10_cell row="0" col="0"/><xacro:rear_marker_id10_cell row="0" col="1"/>
+        <xacro:rear_marker_id10_cell row="0" col="2"/><xacro:rear_marker_id10_cell row="0" col="3"/>
+        <xacro:rear_marker_id10_cell row="0" col="4"/><xacro:rear_marker_id10_cell row="0" col="5"/>
+        <xacro:rear_marker_id10_cell row="1" col="0"/><xacro:rear_marker_id10_cell row="1" col="5"/>
+        <xacro:rear_marker_id10_cell row="2" col="0"/><xacro:rear_marker_id10_cell row="2" col="2"/>
+        <xacro:rear_marker_id10_cell row="2" col="3"/><xacro:rear_marker_id10_cell row="2" col="5"/>
+        <xacro:rear_marker_id10_cell row="3" col="0"/><xacro:rear_marker_id10_cell row="3" col="2"/>
+        <xacro:rear_marker_id10_cell row="3" col="3"/><xacro:rear_marker_id10_cell row="3" col="5"/>
+        <xacro:rear_marker_id10_cell row="4" col="0"/><xacro:rear_marker_id10_cell row="4" col="1"/>
+        <xacro:rear_marker_id10_cell row="4" col="2"/><xacro:rear_marker_id10_cell row="4" col="3"/>
+        <xacro:rear_marker_id10_cell row="4" col="5"/>
+        <xacro:rear_marker_id10_cell row="5" col="0"/><xacro:rear_marker_id10_cell row="5" col="1"/>
+        <xacro:rear_marker_id10_cell row="5" col="2"/><xacro:rear_marker_id10_cell row="5" col="3"/>
+        <xacro:rear_marker_id10_cell row="5" col="4"/><xacro:rear_marker_id10_cell row="5" col="5"/>
+      </xacro:if>
       <collision name="collision">
         <geometry>

Commit message: feat: C1·D435i 선택형 주행과 완주 영상 및 검증 기록 추가

File: src/arena_description/models/arena_car/model.sdf.xacro (robot description, xacro)
@@ -79,4 +79,10 @@
   <xacro:arg name="tof_carrier_size_z" default="0.018"/>
   <xacro:arg name="tof_carrier_mass" default="0.0005"/>
+  <xacro:arg name="tof_front_enabled" default="true"/>
+  <xacro:arg name="tof_front_left_enabled" default="true"/>
+  <xacro:arg name="tof_rear_left_enabled" default="true"/>
+  <xacro:arg name="tof_rear_enabled" default="true"/>
+  <xacro:arg name="tof_rear_right_enabled" default="true"/>
+  <xacro:arg name="tof_front_right_enabled" default="true"/>
   <xacro:arg name="tof_front_pose" default="0.0980 0.0000 0.040 0 0 0"/>
   <xacro:arg name="tof_front_left_pose" default="0.0413 0.0715 0.040 0 0 1.0471975512"/>
@@ -119,4 +125,7 @@
   <xacro:arg name="d435i_depth_cy" default="240.0"/>
   <xacro:arg name="d435i_imu_rate" default="200.0"/>
+  <!-- 검증 영상 전용. 제어 노드는 이 토픽을 구독하지 않습니다. -->
+  <xacro:arg name="chase_camera_enabled" default="false"/>
+  <xacro:arg name="chase_camera_rate" default="20.0"/>
   <xacro:property name="body_length" value="$(arg body_length)"/>
   <xacro:property name="body_width" value="$(arg body_width)"/>
@@ -466,4 +475,28 @@
       <child>d435i_link</child>
     </joint>
+    <!--
+      게임식 3인칭 기록을 위한 1 mg·충돌체 없는 관찰 카메라입니다. 차량과 함께
+      움직이지만 /sim/chase/image는 평가·영상에만 쓰며 자율주행 입력이 아닙니다.
+    -->
+    <xacro:if value="$(arg chase_camera_enabled)">
+      <link name="chase_camera_link">
+        <pose>-0.32 0 0.38 0 0.72 0</pose>
+        <xacro:box_inertial mass="0.000001" x="0.001" y="0.001" z="0.001"/>
+        <sensor name="chase_camera" type="camera">
+          <camera name="chase">
+            <horizontal_fov>1.35</horizontal_fov>
+            <image><width>960</width><height>540</height><format>R8G8B8</format></image>
+            <clip><near>0.05</near><far>30</far></clip>
+          </camera>
+          <always_on>true</always_on>
+          <update_rate>$(arg chase_camera_rate)</update_rate>
+          <visualize>false</visualize>
+          <topic>sim/chase/image</topic>
+        </sensor>
+      </link>
+      <joint name="chase_camera_fixed_joint" type="fixed">
+        <parent>chassis</parent><child>chase_camera_link</child>
+      </joint>
+    </xacro:if>
     <xacro:if value="$(arg lidar_enabled)">
       <link name="lidar_link">
@@ -504,10 +537,10 @@
     </xacro:if>
     <xacro:if value="$(arg tof_enabled)">
-      <xacro:tof_module name="front" pose="$(arg tof_front_pose)" topic="$(arg tof_front_topic)"/>
-      <xacro:tof_module name="front_left" pose="$(arg tof_front_left_pose)" topic="$(arg tof_front_left_topic)"/>
-      <xacro:tof_module name="rear_left" pose="$(arg tof_rear_left_pose)" topic="$(arg tof_rear_left_topic)"/>
-      <xacro:tof_module name="rear" pose="$(arg tof_rear_pose)" topic="$(arg tof_rear_topic)"/>
-      <xacro:tof_module name="rear_right" pose="$(arg tof_rear_right_pose)" topic="$(arg tof_rear_right_topic)"/>
-      <xacro:tof_module name="front_right" pose="$(arg tof_front_right_pose)" topic="$(arg tof_front_right_topic)"/>
+      <xacro:if value="$(arg tof_front_enabled)"><xacro:tof_module name="front" pose="$(arg tof_front_pose)" topic="$(arg tof_front_topic)"/></xacro:if>
+      <xacro:if value="$(arg tof_front_left_enabled)"><xacro:tof_module name="front_left" pose="$(arg tof_front_left_pose)" topic="$(arg tof_front_left_topic)"/></xacro:if>
+      <xacro:if value="$(arg tof_rear_left_enabled)"><xacro:tof_module name="rear_left" pose="$(arg tof_rear_left_pose)" topic="$(arg tof_rear_left_topic)"/></xacro:if>
+      <xacro:if value="$(arg tof_rear_enabled)"><xacro:tof_module name="rear" pose="$(arg tof_rear_pose)" topic="$(arg tof_rear_topic)"/></xacro:if>
+      <xacro:if value="$(arg tof_rear_right_enabled)"><xacro:tof_module name="rear_right" pose="$(arg tof_rear_right_pose)" topic="$(arg tof_rear_right_topic)"/></xacro:if>
+      <xacro:if value="$(arg tof_front_right_enabled)"><xacro:tof_module name="front_right" pose="$(arg tof_front_right_pose)" topic="$(arg tof_front_right_topic)"/></xacro:if>
     </xacro:if>
     <xacro:wheel_link name="front_left_wheel" x="${wheelbase / 2.0}" y="${track_width / 2.0}"/>
